Commit message: updated urdf

File: insertion_robot_description/urdf/insertion_robot.urdf (robot description, URDF)
Before this commit: robot insertion_robot, 7 links, 6 joints
Links:
- added link world
Joints:
- added joint base_fixed_joint: type fixed, parent world, child base_link
- joint base_to_x_axis_joint: limit (none) -> lower=-1 upper=1 effort=1000.0 velocity=0.5; type translational -> prismatic
- joint needle_base_to_needle_joint: limit (none) -> lower=-1.57079 upper=1.57079 effort=1000.0 velocity=0.5; type rotational -> revolute
- joint x_axis_to_y_axis_joint: limit (none) -> lower=-1 upper=1 effort=1000.0 velocity=0.5; type translational -> prismatic
- joint y_axis_to_z_axis_joint: limit (none) -> lower=-1 upper=1 effort=1000.0 velocity=0.5; type translational -> prismatic
- joint z_axis_to_linear_stage_joint: limit (none) -> lower=-1 upper=1 effort=1000.0 velocity=0.5; type translational -> prismatic

Commit message: small sim update

File: insertion_robot_description/urdf/insertion_robot.urdf (robot description, URDF)
Before this commit: robot insertion_robot, 8 links, 7 joints
Links:
- link base_link: mass None -> 10; geometry collision box size=0.2 0.15 0.05; visual box size=0.2 0.15 0.05
- link linear_stage_link: mass None -> 10; geometry collision box size=0.6 0.1 0.2; visual box size=0.6 0.1 0.2
- link needle_base_link: mass None -> 10; geometry collision box size=0.6 0.1 0.2; visual box size=0.6 0.1 0.2
- link needle_link: mass None -> 10; geometry collision box size=0.6 0.1 0.2; visual box size=0.6 0.1 0.2
- link x_axis_link: mass None -> 10; geometry collision box size=0.6 0.1 0.2; visual box size=0.6 0.1 0.2
- link y_axis_link: mass None -> 10; geometry collision box size=0.6 0.1 0.2; visual box size=0.6 0.1 0.2
- link z_axis_link: mass None -> 10; geometry collision box size=0.6 0.1 0.2; visual box size=0.6 0.1 0.2

Commit message: checkpoint

File: insertion_robot_description/urdf/insertion_robot.urdf (robot description, URDF)
Before this commit: robot insertion_robot, 8 links, 7 joints
Links:
- link base_link: mass 10 -> 1
- link linear_stage_link: mass 10 -> 1
- link needle_base_link: mass 10 -> 1
- link needle_link: mass 10 -> 1
- link x_axis_link: mass 10 -> 1
- link y_axis_link: mass 10 -> 1
- link z_axis_link: mass 10 -> 1

Commit message: position controller added

File: insertion_robot_description/urdf/insertion_robot.urdf (robot description, URDF)
Before this commit: robot insertion_robot, 8 links, 7 joints
Joints:
- joint needle_base_to_needle_joint: type revolute -> fixed
